File: board/hdmilight-v3-usb.sch (KiCad schematic (older format))
At the start: 30 parts, among them J1 USB_B_Micro, U2 93CxxB, U3 FT2232D, Y1 6MHz

Commit message: Updated BOM with individual LED colours/types
Parts:
- D1: value LED -> LED Red
- D2: value LED -> LED Green
- Y1: value 6MHz -> 6MHz / 12pF
Changed lines of the file:
@@
 P 7350 4600
 F 0 "D1" H 7341 4816 50  0000 C CNN
-F 1 "LED" H 7341 4725 50  0000 C CNN
+F 1 "LED Red" H 7341 4725 50  0000 C CNN
 F 2 "LED_SMD:LED_0603_1608Metric" H 7350 4600 50  0001 C CNN
 F 3 "~" H 7350 4600 50  0001 C CNN
@@
 P 7350 4900
 F 0 "D2" H 7341 5116 50  0000 C CNN
-F 1 "LED" H 7341 5025 50  0000 C CNN
+F 1 "LED Green" H 7341 5025 50  0000 C CNN
 F 2 "LED_SMD:LED_0603_1608Metric" H 7350 4900 50  0001 C CNN
 F 3 "~" H 7350 4900 50  0001 C CNN
@@
 P 4150 4100
 F 0 "Y1" V 4104 4244 50  0000 L CNN
-F 1 "6MHz" V 4195 4244 50  0000 L CNN
+F 1 "6MHz / 12pF" V 4195 4244 50  0000 L CNN
 F 2 "Crystal:Crystal_SMD_7050-4Pin_7.0x5.0mm" H 4150 4100 50  0001 C CNN
 F 3 "~" H 4150 4100 50  0001 C CNN

Commit message: BOM updates
 * Don't need EEPROM for FTDI
 * Change LED power switching transistor to the one I actually used
 * Sync CSV and interactive BOM files
Parts:
- U2: value 93CxxB -> DNI
Changed lines of the file:
@@
 P 2700 4700
 F 0 "U2" H 2350 4300 50  0000 C CNN
-F 1 "93CxxB" H 2350 4400 50  0000 C CNN
+F 1 "DNI" H 2350 4400 50  0000 C CNN
 F 2 "Package_SO:SOIC-8_3.9x4.9mm_P1.27mm" H 2700 4700 50  0001 C CNN
 F 3 "http://ww1.microchip.com/downloads/en/DeviceDoc/20001749K.pdf" H 2700 4700 50  0001 C CNN
